File: rj11-wemos-hat.kicad_sch (KiCad schematic)
At the start: 24 parts, among them J0 Conn_02x12_Odd_Even, J1 RJ10, J10 SDA, J11 D6, J12 D5, J13 D7, J14 D8, J15 D0, J16 D4, J2 RJ10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

Commit message: Initial version (Revision 1.0)
Parts:
- J0: footprint Connector_PinHeader_2.54mm:PinHeader_2x12_P2.54mm_Vertical -> Connector_PinSocket_2.54mm:PinSocket_2x12_P2.54mm_Vertical
- J10, J11, J12, J13, J14, J15, J16, J6, J7, J8, J9: footprint Connector_Wire:SolderWire-0.15sqmm_1x01_D0.5mm_OD1.5mm -> Chof747 Footprints:Solder Pad 1x1 1.5x3
- JP1, JP2: footprint Connector_PinHeader_2.54mm:PinHeader_1x02_P2.54mm_Vertical -> Chof747 Footprints:Solder Pad 1x2 1.5x3
- SW1: value SW_Push -> RST
- SW2: value SW_Push -> Flash
Changed lines of the file:
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@@
       (effects (font (size 1.27 1.27)))
     )
-    (property "Footprint" "Connector_Wire:SolderWire-0.15sqmm_1x01_D0.5mm_OD1.5mm" (at 109.22 54.61 0)
+    (property "Footprint" "Chof747 Footprints:Solder Pad 1x1 1.5x3" (at 109.22 54.61 0)
       (effects (font (size 1.27 1.27)) hide)
     )
@@
       (effects (font (size 1.27 1.27)))
     )
-    (property "Footprint" "Connector_Wire:SolderWire-0.15sqmm_1x01_D0.5mm_OD1.5mm" (at 109.22 66.04 0)
+    (property "Footprint" "Chof747 Footprints:Solder Pad 1x1 1.5x3" (at 109.22 66.04 0)
       (effects (font (size 1.27 1.27)) hide)
     )
@@
       (effects (font (size 1.27 1.27)))
     )
-    (property "Footprint" "Connector_Wire:SolderWire-0.15sqmm_1x01_D0.5mm_OD1.5mm" (at 109.22 45.72 0)
+    (property "Footprint" "Chof747 Footprints:Solder Pad 1x1 1.5x3" (at 109.22 45.72 0)
       (effects (font (size 1.27 1.27)) hide)
     )
@@
       (effects (font (size 1.27 1.27)))
     )
-    (property "Footprint" "Connector_Wire:SolderWire-0.15sqmm_1x01_D0.5mm_OD1.5mm" (at 109.22 35.56 0)
+    (property "Footprint" "Chof747 Footprints:Solder Pad 1x1 1.5x3" (at 109.22 35.56 0)
       (effects (font (size 1.27 1.27)) hide)
     )
@@
       (effects (font (size 1.27 1.27)))
     )
-    (property "Footprint" "Connector_PinHeader_2.54mm:PinHeader_1x02_P2.54mm_Vertical" (at 133.35 73.66 0)
+    (property "Footprint" "Chof747 Footprints:Solder Pad 1x2 1.5x3" (at 133.35 73.66 0)
       (effects (font (size 1.27 1.27)) hide)
     )
@@
       (effects (font (size 1.27 1.27)))
     )
-    (property "Footprint" "Connector_Wire:SolderWire-0.15sqmm_1x01_D0.5mm_OD1.5mm" (at 109.22 30.48 0)
+    (property "Footprint" "Chof747 Footprints:Solder Pad 1x1 1.5x3" (at 109.22 30.48 0)
       (effects (font (size 1.27 1.27)) hide)
     )
@@
       (effects (font (size 1.27 1.27)))
     )
-    (property "Footprint" "Connector_Wire:SolderWire-0.15sqmm_1x01_D0.5mm_OD1.5mm" (at 109.22 27.94 0)
+    (property "Footprint" "Chof747 Footprints:Solder Pad 1x1 1.5x3" (at 109.22 27.94 0)
       (effects (font (size 1.27 1.27)) hide)
     )
@@
       (effects (font (size 1.27 1.27)))
     )
-    (property "Footprint" "Connector_PinHeader_2.54mm:PinHeader_1x02_P2.54mm_Vertical" (at 133.35 39.37 0)
+    (property "Footprint" "Chof747 Footprints:Solder Pad 1x2 1.5x3" (at 133.35 39.37 0)
       (effects (font (size 1.27 1.27)) hide)
     )
@@
       (effects (font (size 1.27 1.27)) (justify left))
     )
-    (property "Value" "SW_Push" (at 67.31 118.745 90)
+    (property "Value" "Flash" (at 67.31 118.745 90)
       (effects (font (size 1.27 1.27)) (justify left))
     )
@@
       (effects (font (size 1.27 1.27)))
     )
-    (property "Footprint" "Connector_Wire:SolderWire-0.15sqmm_1x01_D0.5mm_OD1.5mm" (at 109.22 63.5 0)
+    (property "Footprint" "Chof747 Footprints:Solder Pad 1x1 1.5x3" (at 109.22 63.5 0)
       (effects (font (size 1.27 1.27)) hide)
     )
@@
       (effects (font (size 1.27 1.27)))
     )
-    (property "Footprint" "Connector_Wire:SolderWire-0.15sqmm_1x01_D0.5mm_OD1.5mm" (at 109.22 68.58 0)
+    (property "Footprint" "Chof747 Footprints:Solder Pad 1x1 1.5x3" (at 109.22 68.58 0)
       (effects (font (size 1.27 1.27)) hide)
     )
@@
       (effects (font (size 1.27 1.27)) (justify left))
     )
-    (property "Value" "SW_Push" (at 43.18 118.745 90)
+    (property "Value" "RST" (at 43.18 118.745 90)
       (effects (font (size 1.27 1.27)) (justify left))
     )
@@
       (effects (font (size 1.27 1.27)))
     )
-    (property "Footprint" "Connector_PinHeader_2.54mm:PinHeader_2x12_P2.54mm_Vertical" (at 48.26 49.53 0)
+    (property "Footprint" "Connector_PinSocket_2.54mm:PinSocket_2x12_P2.54mm_Vertical" (at 48.26 49.53 0)
       (effects (font (size 1.27 1.27)) hide)
     )
@@
       (effects (font (size 1.27 1.27)))
     )
-    (property "Footprint" "Connector_Wire:SolderWire-0.15sqmm_1x01_D0.5mm_OD1.5mm" (at 109.22 48.26 0)
+    (property "Footprint" "Chof747 Footprints:Solder Pad 1x1 1.5x3" (at 109.22 48.26 0)
       (effects (font (size 1.27 1.27)) hide)
     )
@@
       (effects (font (size 1.27 1.27)))
     )
-    (property "Footprint" "Connector_Wire:SolderWire-0.15sqmm_1x01_D0.5mm_OD1.5mm" (at 109.22 38.1 0)
+    (property "Footprint" "Chof747 Footprints:Solder Pad 1x1 1.5x3" (at 109.22 38.1 0)
       (effects (font (size 1.27 1.27)) hide)
     )
@@
       (effects (font (size 1.27 1.27)))
     )
-    (property "Footprint" "Connector_Wire:SolderWire-0.15sqmm_1x01_D0.5mm_OD1.5mm" (at 109.22 57.15 0)
-      (effects (font (size 1.27 1.27)) hide)
-    )
+    (property "Footprint" "Chof747 Footprints:Solder Pad 1x1 1.5x3" (at 109.22 57.15 0)
+      (effects (font (size 1.27 1.27)) hide)
+    )

Commit message: corrected RJ12 socket Connector
Parts:
- J1, J2: symbol Connector:RJ10 -> Chof747 Connectors:RJ12
- J7: value RX -> TX
- J8: value TX -> RX
Connections:
- net GND: now also J1.5, J2.5; no longer J1.4, J2.4
- net PWR_1: now also J1.4; no longer J1.1
- net PWR_2: now also J2.4; no longer J2.1
- net RX: now also J8.1 (Pin_1); no longer J7.1 (Pin_1)
- net TX: now also J7.1 (Pin_1); no longer J8.1 (Pin_1)
Other:
- moved on the sheet: J1, J2
